Commit message: Add files via upload

File: urdf/robot.xacro (robot description, xacro)
@@ -5,5 +5,5 @@
   </gazebo>
   <gazebo reference="left_wheel">
-  		<material> Gazebo/Grey </material>
+  		<material> Gazebo/Red </material>
   </gazebo>
   <gazebo reference="right_wheel">

Commit message: Add files via upload

File: urdf/robot.xacro (robot description, xacro)
@@ -103,3 +103,55 @@
 	<xacro:wheel suffix="left" reflect="1"/>
 	<xacro:wheel suffix="right" reflect="-1"/>
+	<link name="lidar_link">
+    		<xacro:default_inertial mass="0.1"/>
+    		<visual>
+      			<origin xyz="0 0 0" rpy="0 0 0"/>
+      			<geometry>
+        			<cylinder radius="0.04" length="0.02"/>
+      			</geometry>
+      			<material name="blue"/>
+    		</visual>
+    		<collision>
+      			<origin xyz="0 0 0" rpy="0 0 0"/>
+      			<geometry>
+        			<cylinder radius="0.04" length="0.02"/>
+      			</geometry>
+    		</collision>
+  	</link>
+  	<joint name="lidar_joint" type="fixed">
+    		<parent link="base_link"/>
+    		<child link="lidar_link"/>
+    		<origin xyz="0.0 0 0.2" rpy="0 0 0"/>
+  	</joint>
+  	<gazebo reference="lidar_link">
+    		<sensor type="ray" name="laser_sensor">
+      			<pose>0 0 0 0 0 0</pose>
+      			<visualize>true</visualize>
+      			<update_rate>30</update_rate>
+      			<ray>
+        			<scan>
+          				<horizontal>
+            					<samples>360</samples>
+            					<resolution>1</resolution>
+            					<min_angle>-1.5708</min_angle>
+            					<max_angle>1.5708</max_angle>
+          				</horizontal>
+        			</scan>
+        			<range>
+          				<min>0.12</min>
+          				<max>3.5</max>
+          				<resolution>0.01</resolution>
+        			</range>
+        			<noise>
+          				<type>gaussian</type>
+          				<mean>0.0</mean>
+          				<stddev>0.005</stddev>
+        			</noise>
+      			</ray>
+      			<plugin name="gazebo_ros_laser_controller" filename="libgazebo_ros_laser.so">
+        			<topicName>scan</topicName>
+        			<frameName>lidar_link</frameName>
+      			</plugin>
+    		</sensor>
+  	</gazebo>
 </robot>

Commit message: Add files via upload

File: urdf/robot.xacro (robot description, xacro)
@@ -127,5 +127,4 @@
     		<sensor type="ray" name="laser_sensor">
       			<pose>0 0 0 0 0 0</pose>
-      			<visualize>true</visualize>
       			<update_rate>30</update_rate>
       			<ray>
@@ -134,6 +133,6 @@
             					<samples>360</samples>
             					<resolution>1</resolution>
-            					<min_angle>-1.5708</min_angle>
-            					<max_angle>1.5708</max_angle>
+            					<min_angle>-3.1415</min_angle>
+            					<max_angle>3.1415</max_angle>
           				</horizontal>
         			</scan>
@@ -155,3 +154,37 @@
     		</sensor>
   	</gazebo>
+  	<link name="bumper_link">
+    		<xacro:default_inertial mass="0.1"/>
+    		<visual>
+      			<origin xyz="0 0 0" rpy="0 0 0"/>
+      			<geometry>
+        			<box size="0.2 0.05 0.05"/>
+      			</geometry>
+      			<material name="blue"/>
+    		</visual>
+    		<collision>
+      			<origin xyz="0 0 0" rpy="0 0 0"/>
+      			<geometry>
+        			<box size="0.2 0.05 0.05"/>
+      			</geometry>
+    		</collision>
+  	</link>
+  	<joint name="bumper_joint" type="fixed">
+    		<parent link="base_link"/>
+    		<child link="bumper_link"/>
+    		<origin xyz="0.25 0 0.1" rpy="0 0 0"/>
+  	</joint>
+  	<gazebo reference="bumper_link">
+    		<sensor type="contact" name="bumper_sensor">
+      			<always_on>true</always_on>
+      			<update_rate>50</update_rate>
+      			<contact>
+        			<collision>bumper_link</collision>
+      			</contact>
+      			<plugin name="bumper_plugin" filename="libgazebo_ros_bumper.so">
+        			<topicName>bumper</topicName>
+        			<frameName>bumper_link</frameName>
+      			</plugin>
+    		</sensor>
+  	</gazebo>
 </robot>

Commit message: Add controllers

File: urdf/robot.xacro (robot description, xacro)
@@ -183,8 +183,42 @@
       			</contact>
       			<plugin name="bumper_plugin" filename="libgazebo_ros_bumper.so">
-        			<topicName>bumper</topicName>
         			<frameName>bumper_link</frameName>
       			</plugin>
     		</sensor>
   	</gazebo>
+  	<transmission name="trans_left_wheel">
+  		<type>transmission_interface/SimpleTransmission</type>
+  		<joint name="base_left_wheel_joint">
+    			<hardwareInterface>EffortJointInterface</hardwareInterface>
+  		</joint>
+  		<actuator name="left_wheel_motor">
+    			<hardwareInterface>EffortJointInterface</hardwareInterface>
+    			<mechanicalReduction>1</mechanicalReduction>
+  		</actuator>
+	</transmission>
+	<transmission name="trans_right_wheel">
+  		<type>transmission_interface/SimpleTransmission</type>
+  		<joint name="base_right_wheel_joint">
+    			<hardwareInterface>EffortJointInterface</hardwareInterface>
+  		</joint>
+  		<actuator name="right_wheel_motor">
+    			<hardwareInterface>EffortJointInterface</hardwareInterface>
+    			<mechanicalReduction>1</mechanicalReduction>
+  		</actuator>
+	</transmission>
+	<transmission name="trans_caster">
+  		<type>transmission_interface/SimpleTransmission</type>
+  		<joint name="caster_joint">
+    			<hardwareInterface>EffortJointInterface</hardwareInterface>
+  		</joint>
+  		<actuator name="caster_motor">
+    			<hardwareInterface>EffortJointInterface</hardwareInterface>
+    			<mechanicalReduction>1</mechanicalReduction>
+  		</actuator>
+	</transmission>
+	<gazebo>
+  		<plugin name="gazebo_ros_control" filename="libgazebo_ros_control.so">
+    			<robotNamespace>/</robotNamespace>
+  		</plugin>
+	</gazebo>
 </robot>

Commit message: Add files via upload

File: urdf/robot.xacro (robot description, xacro)
@@ -41,4 +41,5 @@
 			<parent link="base_link" />
 			<child link="${suffix}_wheel" />
+			<dynamics damping="0.2" friction="0.1"/>
 		</joint>
 	</xacro:macro>
@@ -79,4 +80,5 @@
 		<parent link="abc"/>
 		<child link="caster"/>
+		<dynamics damping="0.05" friction="0.02"/>
 	</joint>
 	<link name="abc">

Commit message: Add files via upload

File: urdf/robot.xacro (robot description, xacro)
@@ -97,9 +97,10 @@
 		</collision>
 	</link>
-	<joint name="base_abc_joint" type="continuous">
+	<joint name="base_abc_joint" type="revolute">
 		<origin xyz="0.15 0 -0.02" rpy="0 0 0" />
 		<axis xyz="0 0 1" />
 		<parent link="base_link" />
 		<child link="abc" />
+		<limit effort="10" velocity="1.0" lower="-1.57" upper="1.57"/>
 	</joint>
 	<xacro:wheel suffix="left" reflect="1"/>
@@ -224,3 +225,13 @@
   		</plugin>
 	</gazebo>
+	<transmission name="trans_front_wheel">
+  		<type>transmission_interface/SimpleTransmission</type>
+  		<joint name="base_abc_joint">
+    			<hardwareInterface>EffortJointInterface</hardwareInterface>
+  		</joint>
+  		<actuator name="front_wheel_motor">
+    			<hardwareInterface>EffortJointInterface</hardwareInterface>
+    			<mechanicalReduction>1.0</mechanicalReduction>
+  		</actuator>
+	</transmission>
 </robot>

Commit message: Add files via upload

File: urdf/robot.xacro (robot description, xacro)
@@ -111,5 +111,5 @@
       			<origin xyz="0 0 0" rpy="0 0 0"/>
       			<geometry>
-        			<cylinder radius="0.04" length="0.02"/>
+        			<cylinder radius="0.04" length="0.05"/>
       			</geometry>
       			<material name="blue"/>
@@ -118,5 +118,5 @@
       			<origin xyz="0 0 0" rpy="0 0 0"/>
       			<geometry>
-        			<cylinder radius="0.04" length="0.02"/>
+        			<cylinder radius="0.04" length="0.05"/>
       			</geometry>
     		</collision>
@@ -125,5 +125,5 @@
     		<parent link="base_link"/>
     		<child link="lidar_link"/>
-    		<origin xyz="0.0 0 0.2" rpy="0 0 0"/>
+    		<origin xyz="0.0 0 0.22" rpy="0 0 0"/>
   	</joint>
   	<gazebo reference="lidar_link">

Commit message: Add files via upload

File: urdf/robot.xacro (robot description, xacro)
@@ -166,5 +166,5 @@
       			<material name="blue"/>
     		</visual>
-    		<collision>
+    		<collision name="bumper_collision">
       			<origin xyz="0 0 0" rpy="0 0 0"/>
       			<geometry>
@@ -179,15 +179,20 @@
   	</joint>
   	<gazebo reference="bumper_link">
-    		<sensor type="contact" name="bumper_sensor">
-      			<always_on>true</always_on>
-      			<update_rate>50</update_rate>
-      			<contact>
-        			<collision>bumper_link</collision>
-      			</contact>
-      			<plugin name="bumper_plugin" filename="libgazebo_ros_bumper.so">
-        			<frameName>bumper_link</frameName>
-      			</plugin>
-    		</sensor>
-  	</gazebo>
+  		<sensor type="contact" name="bumper_sensor">
+    			<always_on>true</always_on>
+    			<update_rate>50</update_rate>
+    			<contact>
+      				<collision>bumper_collision</collision>
+    			</contact>
+    			<plugin name="bumper_plugin" filename="libgazebo_ros_bumper.so">
+      				<alwaysOn>true</alwaysOn>
+      				<updateRate>50.0</updateRate>
+      				<robotNamespace>/</robotNamespace>
+      				<bodyName>bumper_link</bodyName>
+      				<topicName>bumper_sensor</topicName>
+      				<frameName>bumper_link</frameName>
+    			</plugin>
+  		</sensor>
+	</gazebo>
   	<transmission name="trans_left_wheel">
   		<type>transmission_interface/SimpleTransmission</type>
